File: Schematics/techin514_final_sensor_pcb.kicad_sch (KiCad schematic)
At the start: 11 parts, among them J1 SMD Grove, M1 Stepper_Motor_unipolar_5pin, SW1 SW_Push, SW2 SW_Push, U1 ESP32-C3-XIAO, U2 ESP32-C3-XIAO, U3 SSD1306 OLED, U4 ULN2003

Commit message: Add files via upload
Parts:
- removed M1: Stepper_Motor_unipolar_5pin, symbol Motor:Stepper_Motor_unipolar_5pin
- removed SW1: SW_Push, symbol Switch:SW_Push
- removed U3: SSD1306 OLED, Package_LGA:LGA-14_3x5mm_P0.8mm_LayoutBorder1x6y, symbol Sensor_Motion:ADXL343
- removed U4: ULN2003, symbol Transistor_Array:ULN2003
- added Brd1: SSD1306, SSD1306:128x64OLED, symbol SSD1306-128x64_OLED:SSD1306
- added M1: Stepper_Motor_bipolar, x27_stepper:x27_stepper_two_holes, symbol Motor:Stepper_Motor_bipolar
- added SW2: SW_Push, Button_Switch_THT:SW_PUSH_6mm, symbol Switch:SW_Push
- BT1, BT2: footprint (none) -> Connector_JST:JST_PH_B2B-PH-K_1x02_P2.00mm_Vertical
- D1: footprint (none) -> LED_THT:LED_Rectangular_W5.0mm_H2.0mm-3Pins
- J1: footprint Grove - GSR v1.2:4P-SMD-2.0 -> Connector:NS-Tech_Grove_1x04_P2mm_Vertical
- SW1: renamed from SW2; footprint (none) -> Button_Switch_THT:SW_PUSH_6mm
- U1, U2: footprint RF_Module:ESP32-C3-DevKitM-1 -> esp32c3:XIAO_ESP32; symbol RF_Module:ESP32-C3-DevKitM-1 -> GIX_ESP32:XIAO_ESP32
Connections:
- net GND: now also U1.13 (GND), U2.13 (GND), Brd1.1 (GND); no longer U1.21 (GND), U2.21 (GND)
- net SIG: now also U2.1 (GPIO1_A0_D0); no longer U2.9 (D0)
- net -BATT: now reaches BT1.2 (-)
- net -BATT: now also U1.16 (-BATT); no longer U1.17 (BAT-)
- net +BATT: now reaches SW1.1
- net +BATT: now also U1.15 (+BATT); no longer U1.18 (BAT+)
- net at BT2.1 (+): now also SW2.2
- net -BATT_S: now reaches BT2.2 (-)
- net -BATT_S: now also U2.16 (-BATT); no longer U2.17 (BAT-)
- net at U1.3 (GPIO3_A2_D2): now also M1.3
- net at U1.4 (GPIO4_A3_D3): now also M1.4
- net at U1.5 (GPIO4_A3_D3_SDA): now also Brd1.4 (SDA)
- removed net VCC: D1.3 (VDD), J1.3, U1.22 (3V3), U2.22 (3V3)
- new net: Brd1.3 (SCL), U1.6 (GPIO6_A5_D5_SCL)
- new net: M1.2 (-), U1.1 (GPIO1_A0_D0)
- new net: M1.1, U1.2 (GPIO2_A1_D1)
- new net +BATT_S: SW2.1, U2.15 (+BATT)
- new net 3V3: Brd1.2 (VCC), D1.3 (VDD), U1.12 (3V3)
- new net 3V3_S: J1.3, U2.12 (3V3)
- now unconnected: U1.8 (GND), U2.6 (GND), U2.8 (GND)
Other:
- title: (none) -> SuHyunJung_Final Project
- moved on the sheet: BT1, D1, SW1
